File: keyboard.kicad_sch (KiCad schematic)
At the start: 6 parts, among them J3 USB_A

Commit message: HW Rev 1.0
Parts:
- renumbered J3 to USB2
Other:
- note added: "Keyboard"
- moved on the sheet: C31, D6, D7, R45, R46, USB2
