File: rp2040.kicad_sch (KiCad schematic)
At the start: 28 parts, among them SW1 Flash Button, U1 RP2040, U2 W25Q128JVS, Y1 ABM8-272-T3

Commit message: HW Rev 1.0
Parts:
- renumbered U2 to FL1, U1 to RP1
Other:
- note added: "Flash"
- note added: "LED"
- note added: "RP2040"
- moved on the sheet: C1, C10, C11, C12, C13, C14, C2, C3, C4, C5, C6, C7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
