File: composite.kicad_sch (KiCad schematic)
At the start: 16 parts

Commit message: Updated HW
Parts:
- R43: renamed from R45; footprint Resistor_SMD:R_0805_2012Metric_Pad1.20x1.40mm_HandSolder -> LIBS:Medved_R_0805
- R44: renamed from R46; footprint Resistor_SMD:R_0805_2012Metric_Pad1.20x1.40mm_HandSolder -> LIBS:Medved_R_0805
- R45: renamed from R47; footprint Resistor_SMD:R_0805_2012Metric_Pad1.20x1.40mm_HandSolder -> LIBS:Medved_R_0805
- R46: renamed from R48; footprint Resistor_SMD:R_0805_2012Metric_Pad1.20x1.40mm_HandSolder -> LIBS:Medved_R_0805
- R47: renamed from R49; footprint Resistor_SMD:R_0805_2012Metric_Pad1.20x1.40mm_HandSolder -> LIBS:Medved_R_0805
- R48: renamed from R50; footprint Resistor_SMD:R_0805_2012Metric_Pad1.20x1.40mm_HandSolder -> LIBS:Medved_R_0805
- R49: renamed from R51; footprint Resistor_SMD:R_0805_2012Metric_Pad1.20x1.40mm_HandSolder -> LIBS:Medved_R_0805
- R50: renamed from R52; footprint Resistor_SMD:R_0805_2012Metric_Pad1.20x1.40mm_HandSolder -> LIBS:Medved_R_0805
- R51: renamed from R53; footprint Resistor_SMD:R_0805_2012Metric_Pad1.20x1.40mm_HandSolder -> LIBS:Medved_R_0805
- R52: renamed from R54; footprint Resistor_SMD:R_0805_2012Metric_Pad1.20x1.40mm_HandSolder -> LIBS:Medved_R_0805
- R53: renamed from R55; footprint Resistor_SMD:R_0805_2012Metric_Pad1.20x1.40mm_HandSolder -> LIBS:Medved_R_0805
- R54: renamed from R56; footprint Resistor_SMD:R_0805_2012Metric_Pad1.20x1.40mm_HandSolder -> LIBS:Medved_R_0805
- R55: renamed from R57; footprint Resistor_SMD:R_0805_2012Metric_Pad1.20x1.40mm_HandSolder -> LIBS:Medved_R_0805
- R56: renamed from R58; footprint Resistor_SMD:R_0805_2012Metric_Pad1.20x1.40mm_HandSolder -> LIBS:Medved_R_0805
- renumbered C30 to C17

Commit message: HW Rev 2.0
Other:
- title: Mini FRANK -> FRANK
Changed lines of the file:
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@@
 	(generator "eeschema")
 	(generator_version "8.0")
-	(paper "A3")
+	(paper "A4")
 	(title_block
-		(title "Mini FRANK")
-		(date "2024-11-13")
-		(rev "1.2")
+		(title "FRANK")
+		(date "2024-12-15")
+		(rev "2.0")
 		(company "Mikhail Matveev")
-		(comment 1 "https://github.com/xtremespb/minifrank")
+		(comment 1 "https://github.com/xtremespb/frank2")
 	)
 	(junction
