File: frank2.kicad_sch (KiCad schematic)
At the start: 4 parts, among them J1 USB Data, J2 Keyboard Data

Commit message: HW Rev 1.0
Parts:
- J1: footprint Connector_PinHeader_2.54mm:PinHeader_2x02_P2.54mm_Vertical -> LIBS:Medved_2x02
- J2: footprint Connector_PinHeader_2.54mm:PinHeader_1x02_P2.54mm_Vertical -> LIBS:Medved_PinHeader_1x02
Other:
- note added: "Power LED"
- note added: "USB Connection Switch"
- moved on the sheet: J1, J2, L1, R1

Commit message: Updated HW
Parts:
- removed J1: USB Data, LIBS:Medved_2x02, symbol Connector_Generic:Conn_02x02_Odd_Even
- removed J2: Keyboard Data, LIBS:Medved_PinHeader_1x02, symbol Connector:Conn_01x02_Pin
- removed L1: LED, LED_SMD:LED_0805_2012Metric_Pad1.15x1.40mm_HandSolder, symbol Device:LED
- removed R1: 10K, Resistor_SMD:R_0805_2012Metric_Pad1.20x1.40mm_HandSolder, symbol Device:R
- added H1, H2, H3, H4: MountingHole, LIBS:Medved_MountingHole_V2, symbol Mechanical:MountingHole
Connections:
- no-connect marks 5 -> 18
Other:
- removed sheet Keyboard
- removed sheet RP2040
- removed sheet Reset
- added sheet Composite Video (composite.kicad_sch)
- added sheet PS2 (ps2.kicad_sch)
- added sheet Pico (pico1.kicad_sch)
- added sheet USB Stacked (usbstack.kicad_sch)
- added sheet Zero (zero.kicad_sch)
- note removed: "Power LED"
- note removed: "USB Connection Switch"

Commit message: HW Rev 2.0
Other:
- title: FRANK2 -> FRANK
Changed lines of the file:
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@@
 	(paper "A4")
 	(title_block
-		(title "FRANK2")
-		(date "2024-11-21")
-		(rev "1.0")
+		(title "FRANK")
+		(date "2024-12-15")
+		(rev "2.0")
 		(company "Mikhail Matveev")
 		(comment 1 "https://github.com/xtremespb/frank2")
