File: gamepad.kicad_sch (KiCad schematic)
At the start: 4 parts

Commit message: HW Rev 1.0
Parts:
- JOY1: renamed from DB1; footprint Connector_Dsub:DSUB-9_Male_Horizontal_P2.77x2.84mm_EdgePinOffset4.94mm_Housed_MountingHolesOffset7.48mm -> LIBS:DB9
Other:
- note added: "Gamepad"
- moved on the sheet: D1, JOY1, JP1, R11

Commit message: Updated HW
Parts:
- D1: footprint Diode_SMD:D_0805_2012Metric_Pad1.15x1.40mm_HandSolder -> LIBS:Medved_D_0805
- R1: renamed from R11; footprint Resistor_SMD:R_0805_2012Metric_Pad1.20x1.40mm_HandSolder -> LIBS:Medved_R_0805
Changed lines of the file:
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@@
 		(on_board yes)
 		(dnp no)
-		(property "Reference" "#PWR019"
+		(property "Reference" "#PWR01"
 			(at 63.5 76.2 0)
 			(effects
@@
 			(project "frank2"
 				(path "/8c0b3d8b-46d3-4173-ab1e-a61765f77d61/48d67e7d-16ec-4bee-8dad-45e13f9405cf"
-					(reference "#PWR019")
-					(unit 1)
-				)
-				(path "/8c0b3d8b-46d3-4173-ab1e-a61765f77d61/5c27e917-1b31-4eec-8dee-943d0b3ebe85"
-					(reference "#PWR047")
+					(reference "#PWR01")
+					(unit 1)
+				)
+				(path "/8c0b3d8b-46d3-4173-ab1e-a61765f77d61/5c27e917-1b31-4eec-8dee-943d0b3ebe85"
+					(reference "#PWR026")
 					(unit 1)
 				)
@@
 			)
 		)
-		(property "Footprint" "Diode_SMD:D_0805_2012Metric_Pad1.15x1.40mm_HandSolder"
+		(property "Footprint" "LIBS:Medved_D_0805"
 			(at 63.5 64.77 0)
 			(effects
@@
 		(dnp no)
 		(fields_autoplaced yes)
-		(property "Reference" "#PWR020"
+		(property "Reference" "#PWR02"
 			(at 76.2 58.42 0)
 			(effects
@@
 			(project ""
 				(path "/8c0b3d8b-46d3-4173-ab1e-a61765f77d61/48d67e7d-16ec-4bee-8dad-45e13f9405cf"
-					(reference "#PWR020")
-					(unit 1)
-				)
-				(path "/8c0b3d8b-46d3-4173-ab1e-a61765f77d61/5c27e917-1b31-4eec-8dee-943d0b3ebe85"
-					(reference "#PWR048")
+					(reference "#PWR02")
+					(unit 1)
+				)
+				(path "/8c0b3d8b-46d3-4173-ab1e-a61765f77d61/5c27e917-1b31-4eec-8dee-943d0b3ebe85"
+					(reference "#PWR027")
 					(unit 1)
 				)
@@
 		(dnp no)
 		(fields_autoplaced yes)
-		(property "Reference" "#PWR021"
+		(property "Reference" "#PWR03"
 			(at 71.12 52.07 0)
 			(effects
@@
 			(project ""
 				(path "/8c0b3d8b-46d3-4173-ab1e-a61765f77d61/48d67e7d-16ec-4bee-8dad-45e13f9405cf"
-					(reference "#PWR021")
-					(unit 1)
-				)
-				(path "/8c0b3d8b-46d3-4173-ab1e-a61765f77d61/5c27e917-1b31-4eec-8dee-943d0b3ebe85"
-					(reference "#PWR049")
+					(reference "#PWR03")
+					(unit 1)
+				)
+				(path "/8c0b3d8b-46d3-4173-ab1e-a61765f77d61/5c27e917-1b31-4eec-8dee-943d0b3ebe85"
+					(reference "#PWR028")
 					(unit 1)
 				)
@@
 		(on_board yes)
 		(dnp no)
-		(property "Reference" "R11"
+		(property "Reference" "R1"
 			(at 66.04 57.15 90)
 			(effects
@@
 			)
 		)
-		(property "Footprint" "Resistor_SMD:R_0805_2012Metric_Pad1.20x1.40mm_HandSolder"
+		(property "Footprint" "LIBS:Medved_R_0805"
 			(at 68.58 61.468 90)
 			(effects
@@
 			(project "frank2"
 				(path "/8c0b3d8b-46d3-4173-ab1e-a61765f77d61/48d67e7d-16ec-4bee-8dad-45e13f9405cf"
-					(reference "R11")
-					(unit 1)
-				)
-				(path "/8c0b3d8b-46d3-4173-ab1e-a61765f77d61/5c27e917-1b31-4eec-8dee-943d0b3ebe85"
-					(reference "R34")
-					(unit 1)
-				)
+					(reference "R1")
+					(unit 1)
+				)
+				(path "/8c0b3d8b-46d3-4173-ab1e-a61765f77d61/5c27e917-1b31-4eec-8dee-943d0b3ebe85"
+					(reference "R24")
+					(unit 1)
+				)

Commit message: HW Rev 2.0
Other:
- title: FRANK2 -> FRANK
Changed lines of the file:
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@@
 	(paper "A4")
 	(title_block
-		(title "FRANK2")
-		(date "2024-11-21")
-		(rev "1.0")
+		(title "FRANK")
+		(date "2024-12-15")
+		(rev "2.0")
 		(company "Mikhail Matveev")
 		(comment 1 "https://github.com/xtremespb/frank2")
