File: pico1.kicad_sch (KiCad schematic)
At the start: 1 part

Commit message: HW Rev 2.0
Other:
- title: FRANK2 -> FRANK
Changed lines of the file:
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@@
 	(paper "A4")
 	(title_block
-		(title "FRANK2")
-		(date "2024-11-21")
-		(rev "1.0")
+		(title "FRANK")
+		(date "2024-12-15")
+		(rev "2.0")
 		(company "Mikhail Matveev")
 		(comment 1 "https://github.com/xtremespb/frank2")
