File: power.kicad_sch (KiCad schematic)
At the start: 8 parts, among them U3 NCP1117-3.3_SOT223

Commit message: HW Rev 1.0
Parts:
- renumbered U3 to U1
Other:
- note added: "Power Input"
- note added: "Power LED (+3V)"
- moved on the sheet: C15, C16, L3, R12, R13, R14, U1

Commit message: Updated HW
Parts:
- removed C16: 10u, Capacitor_SMD:C_0805_2012Metric_Pad1.18x1.45mm_HandSolder, symbol Device:C
- removed U1: NCP1117-3.3_SOT223, Package_TO_SOT_SMD:SOT-223-3_TabPin2, symbol Regulator_Linear:NCP1117-3.3_SOT223
- C1: renamed from C15; footprint Capacitor_SMD:C_0805_2012Metric_Pad1.18x1.45mm_HandSolder -> LIBS:Medved_C_0805
- L1: renamed from L3; value LED -> GREEN; footprint LED_SMD:LED_0805_2012Metric_Pad1.15x1.40mm_HandSolder -> LIBS:Medved_L_0805
- R2: renamed from R12; footprint Resistor_SMD:R_0805_2012Metric_Pad1.20x1.40mm_HandSolder -> LIBS:Medved_R_0805
- R3: renamed from R13; footprint Resistor_SMD:R_0805_2012Metric_Pad1.20x1.40mm_HandSolder -> LIBS:Medved_R_0805
- R4: renamed from R14; footprint Resistor_SMD:R_0805_2012Metric_Pad1.20x1.40mm_HandSolder -> LIBS:Medved_R_0805

Commit message: HW Rev 2.0
Other:
- title: FRANK2 -> FRANK
Changed lines of the file:
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@@
 	(paper "A4")
 	(title_block
-		(title "FRANK2")
-		(date "2024-11-21")
-		(rev "1.0")
+		(title "FRANK")
+		(date "2024-12-15")
+		(rev "2.0")
 		(company "Mikhail Matveev")
 		(comment 1 "https://github.com/xtremespb/frank2")
