File: ps2.kicad_sch (KiCad schematic)
At the start: 8 parts

Commit message: Updated HW
Parts:
- added C16: 0.1u, LIBS:Medved_C_0805, symbol Device:C
- added D6, D7: 3V3, LIBS:Medved_D_0805, symbol Device:D_Zener
- added JP6, JP7: RP ZERO +5V Jumper, LIBS:Medved_PinHeader_1x02_P2.54mm_Vertical_R, symbol Jumper:Jumper_2_Bridged
- added R35, R40: 1k, LIBS:Medved_R_0805, symbol Device:R
- added R36, R37: 100R, LIBS:Medved_R_0805, symbol Device:R
- C15: renamed from C25; footprint Capacitor_SMD:C_0805_2012Metric_Pad1.18x1.45mm_HandSolder -> LIBS:Medved_C_0805
- D8: renamed from D3; footprint LIBS:R_0805_PLUS -> LIBS:Medved_D_0805
- D9: renamed from D4; footprint LIBS:R_0805_PLUS -> LIBS:Medved_D_0805
- R38: renamed from R33; footprint Resistor_SMD:R_0805_2012Metric_Pad1.20x1.40mm_HandSolder -> LIBS:Medved_R_0805
- R39: renamed from R34; footprint Resistor_SMD:R_0805_2012Metric_Pad1.20x1.40mm_HandSolder -> LIBS:Medved_R_0805
- R41: renamed from R35; footprint Resistor_SMD:R_0805_2012Metric_Pad1.20x1.40mm_HandSolder -> LIBS:Medved_R_0805
- R42: renamed from R36; footprint Resistor_SMD:R_0805_2012Metric_Pad1.20x1.40mm_HandSolder -> LIBS:Medved_R_0805
Connections:
- net GND: now also C16.2, D6.2 (A), D7.2 (A)
- net VBUS: now also C16.1, R35.1, R40.1
- net PS/2 MDATA: now reaches KB1.2
- net PS/2 MDATA: now also R35.2, R36.1
- net PS/2 MCLK: now reaches KB1.6
- net PS/2 MCLK: now also R37.1, R40.2
- net PS/2 CLK renamed PS/2 KCLK
- net PS/2 DATA renamed PS/2 KDATA
- new net: D6.1 (K), JP6.2 (B), R36.2
- new net: D7.1 (K), JP7.1 (A), R37.2
- new net GPIO14: JP7.2 (B)
- new net GPIO15: JP6.1 (A)
- no-connect marks 2 -> 0

Commit message: HW Rev 2.0
Other:
- title: Mini FRANK -> FRANK
Changed lines of the file:
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@@
 	(generator "eeschema")
 	(generator_version "8.0")
-	(paper "A3")
+	(paper "A4")
 	(title_block
-		(title "Mini FRANK")
-		(date "2024-11-13")
-		(rev "1.2")
+		(title "FRANK")
+		(date "2024-12-15")
+		(rev "2.0")
 		(company "Mikhail Matveev")
-		(comment 1 "https://github.com/xtremespb/minifrank")
+		(comment 1 "https://github.com/xtremespb/frank2")
 	)
 	(junction
