File: psram.kicad_sch (KiCad schematic)
At the start: 3 parts

Commit message: HW Rev 1.0
Parts:
- added JP6, JP7: RP ZERO +5V Jumper, LIBS:Medved_PinHeader_1x02_P2.54mm_Vertical_R, symbol Jumper:Jumper_2_Bridged
Connections:
- net GPIO18: now also JP6.2 (B); no longer PSR1.1 (~{CE})
- net GPIO19: now also JP7.1 (A); no longer PSR1.6 (SCLK)
- new net: JP6.1 (A), PSR1.1 (~{CE})
- new net: JP7.2 (B), PSR1.6 (SCLK)
Other:
- note added: "PSRAM"
- moved on the sheet: C30, JP8, PSR1

Commit message: Updated HW
Parts:
- C18: renamed from C30; footprint Capacitor_SMD:C_0805_2012Metric_Pad1.18x1.45mm_HandSolder -> LIBS:Medved_C_0805
- renumbered JP8 to JP10, JP6 to JP8, JP7 to JP9
Changed lines of the file:
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@@
-		)
-	)
-	(label "+3V3"
-		(at 67.31 40.64 0)
-		(fields_autoplaced yes)
-		(effects
-			(font
-				(size 1.27 1.27)
-			)
-			(justify left bottom)
 		)
 	)
@@
 		(on_board yes)
 		(dnp no)
-		(property "Reference" "JP6"
+		(property "Reference" "JP8"
 			(at 90.17 43.18 0)
 			(effects
@@
 			(project "frank2"
 				(path "/8c0b3d8b-46d3-4173-ab1e-a61765f77d61/cfde7a60-7ac3-405d-8b86-f95521b6825b"
-					(reference "JP6")
+					(reference "JP8")
 					(unit 1)
 				)
@@
 		(on_board yes)
 		(dnp no)
-		(property "Reference" "#PWR057"
+		(property "Reference" "#PWR045"
 			(at 62.23 72.39 0)
 			(effects
@@
 			(project "frank2"
 				(path "/8c0b3d8b-46d3-4173-ab1e-a61765f77d61/cfde7a60-7ac3-405d-8b86-f95521b6825b"
-					(reference "#PWR057")
+					(reference "#PWR045")
 					(unit 1)
 				)
@@
 		(on_board yes)
 		(dnp no)
-		(property "Reference" "JP7"
+		(property "Reference" "JP9"
 			(at 90.17 50.8 0)
 			(effects
@@
 			(project "frank2"
 				(path "/8c0b3d8b-46d3-4173-ab1e-a61765f77d61/cfde7a60-7ac3-405d-8b86-f95521b6825b"
-					(reference "JP7")
+					(reference "JP9")
+					(unit 1)
+				)
+			)
+		)
+	)
+	(symbol
+		(lib_id "power:+3V3")
+		(at 72.39 40.64 0)
+		(unit 1)
+		(exclude_from_sim no)
+		(in_bom yes)
+		(on_board yes)
+		(dnp no)
+		(fields_autoplaced yes)
+		(property "Reference" "#PWR067"
+			(at 72.39 44.45 0)
+			(effects
+				(font
+					(size 1.27 1.27)
+				)
+				(hide yes)
+			)
+		)
+		(property "Value" "+3V3"
+			(at 72.39 35.56 0)
+			(effects
+				(font
+					(size 1.27 1.27)
+				)
+			)
+		)
+		(property "Footprint" ""
+			(at 72.39 40.64 0)
+			(effects
+				(font
+					(size 1.27 1.27)
+				)
+				(hide yes)
+			)
+		)
+		(property "Datasheet" ""
+			(at 72.39 40.64 0)
+			(effects
+				(font
+					(size 1.27 1.27)
+				)
+				(hide yes)
+			)
+		)
+		(property "Description" "Power symbol creates a global label with name \"+3V3\""
+			(at 72.39 40.64 0)
+			(effects
+				(font
+					(size 1.27 1.27)
+				)
+				(hide yes)
+			)
+		)
+		(pin "1"
+		)
+		(instances
+			(project ""
+				(path "/8c0b3d8b-46d3-4173-ab1e-a61765f77d61/cfde7a60-7ac3-405d-8b86-f95521b6825b"
+					(reference "#PWR067")
 					(unit 1)
 				)
@@
 		(on_board yes)
 		(dnp no)
-		(property "Reference" "C30"
+		(property "Reference" "C18"
 			(at 44.831 47.0916 0)
 			(effects
@@
 			)
 		)
-		(property "Footprint" "Capacitor_SMD:C_0805_2012Metric_Pad1.18x1.45mm_HandSolder"
+		(property "Footprint" "LIBS:Medved_C_0805"
 			(at 42.8752 52.07 0)
 			(effects
@@
 			(project "frank2"
 				(path "/8c0b3d8b-46d3-4173-ab1e-a61765f77d61/cfde7a60-7ac3-405d-8b86-f95521b6825b"
-					(reference "C30")
+					(reference "C18")
 					(unit 1)
 				)
@@
 		(on_board yes)
 		(dnp no)
-		(property "Reference" "JP8"
+		(property "Reference" "JP10"
 			(at 91.44 64.77 0)
 			(effects
@@
 			(project "frank2"
 				(path "/8c0b3d8b-46d3-4173-ab1e-a61765f77d61/cfde7a60-7ac3-405d-8b86-f95521b6825b"
-					(reference "JP8")
+					(reference "JP10")
 					(unit 1)
 				)
@@
 		(on_board yes)
 		(dnp no)
-		(property "Reference" "#PWR056"
+		(property "Reference" "#PWR044"
 			(at 41.91 62.23 0)
 			(effects
@@
 			(project "frank2"
 				(path "/8c0b3d8b-46d3-4173-ab1e-a61765f77d61/cfde7a60-7ac3-405d-8b86-f95521b6825b"
-					(reference "#PWR056")
-					(unit 1)
-				)
+					(reference "#PWR044")
+					(unit 1)
+				)

Commit message: HW Rev 2.0
Other:
- title: FRANK2 -> FRANK
Changed lines of the file:
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@@
 	(paper "A4")
 	(title_block
-		(title "FRANK2")
-		(date "2024-11-21")
-		(rev "1.0")
+		(title "FRANK")
+		(date "2024-12-15")
+		(rev "2.0")
 		(company "Mikhail Matveev")
 		(comment 1 "https://github.com/xtremespb/frank2")
