File: sd.kicad_sch (KiCad schematic)
At the start: 2 parts

Commit message: HW Rev 1.0
Other:
- note added: "Micro SD Card"
- moved on the sheet: C18, SD1
Changed lines of the file:
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@@
 	(generator "eeschema")
 	(generator_version "8.0")
-	(paper "A3")
+	(paper "A4")
 	(title_block
 		(title "FRANK2")
@@
 	)
 	(no_connect
-		(at 55.88 63.5)
+		(at 68.58 67.31)
 	)
 	(no_connect
-		(at 55.88 45.72)
+		(at 68.58 49.53)
 	)
 	(no_connect
-		(at 99.06 68.58)
-	)
-	(wire
-		(pts
-			(xy 22.86 58.42) (xy 55.88 58.42)
-		)
-		(stroke
-			(width 0)
-			(type default)
-		)
-	)
-	(wire
-		(pts
-			(xy 22.86 46.99) (xy 22.86 53.34)
-		)
-		(stroke
-			(width 0)
-			(type default)
-		)
-	)
-	(wire
-		(pts
-			(xy 22.86 58.42) (xy 22.86 67.31)
-		)
-		(stroke
-			(width 0)
-			(type default)
-		)
-	)
-	(wire
-		(pts
-			(xy 43.18 60.96) (xy 55.88 60.96)
-		)
-		(stroke
-			(width 0)
-			(type default)
-		)
-	)
-	(wire
-		(pts
-			(xy 43.18 50.8) (xy 55.88 50.8)
-		)
-		(stroke
-			(width 0)
-			(type default)
-		)
-	)
-	(wire
-		(pts
-			(xy 43.18 55.88) (xy 55.88 55.88)
-		)
-		(stroke
-			(width 0)
-			(type default)
-		)
-	)
-	(wire
-		(pts
-			(xy 43.18 48.26) (xy 55.88 48.26)
-		)
-		(stroke
-			(width 0)
-			(type default)
-		)
-	)
-	(wire
-		(pts
-			(xy 22.86 53.34) (xy 55.88 53.34)
-		)
-		(stroke
-			(width 0)
-			(type default)
+		(at 111.76 72.39)
+	)
+	(wire
+		(pts
+			(xy 35.56 62.23) (xy 68.58 62.23)
+		)
+		(stroke
+			(width 0)
+			(type default)
+		)
+	)
+	(wire
+		(pts
+			(xy 35.56 50.8) (xy 35.56 57.15)
+		)
+		(stroke
+			(width 0)
+			(type default)
+		)
+	)
+	(wire
+		(pts
+			(xy 35.56 62.23) (xy 35.56 71.12)
+		)
+		(stroke
+			(width 0)
+			(type default)
+		)
+	)
+	(wire
+		(pts
+			(xy 55.88 64.77) (xy 68.58 64.77)
+		)
+		(stroke
+			(width 0)
+			(type default)
+		)
+	)
+	(wire
+		(pts
+			(xy 55.88 54.61) (xy 68.58 54.61)
+		)
+		(stroke
+			(width 0)
+			(type default)
+		)
+	)
+	(wire
+		(pts
+			(xy 55.88 59.69) (xy 68.58 59.69)
+		)
+		(stroke
+			(width 0)
+			(type default)
+		)
+	)
+	(wire
+		(pts
+			(xy 55.88 52.07) (xy 68.58 52.07)
+		)
+		(stroke
+			(width 0)
+			(type default)
+		)
+	)
+	(wire
+		(pts
+			(xy 35.56 57.15) (xy 68.58 57.15)
+		)
+		(stroke
+			(width 0)
+			(type default)
+		)
+	)
+	(text "Micro SD Card"
+		(exclude_from_sim no)
+		(at 124.968 35.56 0)
+		(effects
+			(font
+				(size 2.54 2.54)
+			)
+			(justify left bottom)
 		)
 	)
 	(label "+3V3"
-		(at 49.53 53.34 0)
+		(at 62.23 57.15 0)
 		(fields_autoplaced yes)
 		(effects
@@
 	(hierarchical_label "GPIO2"
 		(shape input)
-		(at 43.18 55.88 180)
+		(at 55.88 59.69 180)
 		(fields_autoplaced yes)
 		(effects
@@
 	(hierarchical_label "GPIO4"
 		(shape input)
-		(at 43.18 60.96 180)
+		(at 55.88 64.77 180)
 		(fields_autoplaced yes)
 		(effects
@@
 	(hierarchical_label "GPIO3"
 		(shape input)
-		(at 43.18 50.8 180)
+		(at 55.88 54.61 180)
 		(fields_autoplaced yes)
 		(effects
@@
 	(hierarchical_label "GPIO5"
 		(shape input)
-		(at 43.18 48.26 180)
+		(at 55.88 52.07 180)
 		(fields_autoplaced yes)
 		(effects
@@
 	(symbol
 		(lib_id "power:GND")
-		(at 22.86 67.31 0)
+		(at 35.56 71.12 0)
 		(unit 1)
 		(exclude_from_sim no)
@@
 		(dnp no)
 		(fields_autoplaced yes)
-		(property "Reference" "#PWR037"
-			(at 22.86 73.66 0)
+		(property "Reference" "#PWR036"
+			(at 35.56 77.47 0)
 			(effects
 				(font
@@
 		)
 		(property "Value" "GND"
-			(at 22.86 71.7534 0)
+			(at 35.56 75.5634 0)
 			(effects
 				(font
@@
 		)
 		(property "Footprint" ""
-			(at 22.86 67.31 0)
+			(at 35.56 71.12 0)
 			(effects
 				(font
@@
 		)
 		(property "Datasheet" ""
-			(at 22.86 67.31 0)
+			(at 35.56 71.12 0)
 			(effects
 				(font
@@
 		)
 		(property "Description" ""
-			(at 22.86 67.31 0)
-			(effects
-				(font
-					(size 1.27 1.27)
-				)
-				(hide yes)
-			)
-		)
-		(pin "1"
-		)
-		(instances
-			(project "frank2"
-				(path "/8c0b3d8b-46d3-4173-ab1e-a61765f77d61/1910744e-2d47-4355-a4aa-76cd3c94388f"
-					(reference "#PWR037")
-					(unit 1)
-				)
-			)
-		)
-	)
-	(symbol
-		(lib_id "power:GND")
-		(at 22.86 39.37 180)
-		(unit 1)
-		(exclude_from_sim no)
-		(in_bom yes)
-		(on_board yes)
-		(dnp no)
-		(property "Reference" "#PWR036"
-			(at 22.86 33.02 0)
-			(effects
-				(font
-					(size 1.27 1.27)
-				)
-				(hide yes)
-			)
-		)
-		(property "Value" "GND"
-			(at 16.51 36.83 0)
-			(effects
-				(font
-					(size 1.27 1.27)
-				)
-				(justify right)
-				(hide yes)
-			)
-		)
-		(property "Footprint" ""
-			(at 22.86 39.37 0)
-			(effects
-				(font
-					(size 1.27 1.27)
-				)
-				(hide yes)
-			)
-		)
-		(property "Datasheet" ""
-			(at 22.86 39.37 0)
-			(effects
-				(font
-					(size 1.27 1.27)
-				)
-				(hide yes)
-			)
-		)
-		(property "Description" ""
-			(at 22.86 39.37 0)
+			(at 35.56 71.12 0)
 			(effects
 				(font
@@
 	)
 	(symbol
+		(lib_id "power:GND")
+		(at 35.56 43.18 180)
+		(unit 1)
+		(exclude_from_sim no)
+		(in_bom yes)
+		(on_board yes)
+		(dnp no)
+		(property "Reference" "#PWR035"
+			(at 35.56 36.83 0)
+			(effects
+				(font
+					(size 1.27 1.27)
+				)
+				(hide yes)
+			)
+		)
+		(property "Value" "GND"
+			(at 29.21 40.64 0)
+			(effects
+				(font
+					(size 1.27 1.27)
+				)
+				(justify right)
+				(hide yes)
+			)
+		)
+		(property "Footprint" ""
+			(at 35.56 43.18 0)
+			(effects
+				(font
+					(size 1.27 1.27)
+				)
+				(hide yes)
+			)
+		)
+		(property "Datasheet" ""
+			(at 35.56 43.18 0)
+			(effects
+				(font
+					(size 1.27 1.27)
+				)
+				(hide yes)
+			)
+		)
+		(property "Description" ""
+			(at 35.56 43.18 0)
+			(effects
+				(font
+					(size 1.27 1.27)
+				)
+				(hide yes)
+			)
+		)
+		(pin "1"
+		)
+		(instances
+			(project "frank2"
+				(path "/8c0b3d8b-46d3-4173-ab1e-a61765f77d61/1910744e-2d47-4355-a4aa-76cd3c94388f"
+					(reference "#PWR035")
+					(unit 1)
+				)
+			)
+		)
+	)
+	(symbol
 		(lib_id "Device:C")
-		(at 22.86 43.18 0)
+		(at 35.56 46.99 0)
 		(unit 1)
 		(exclude_from_sim no)
@@
 		(dnp no)
 		(property "Reference" "C18"
-			(at 25.781 42.0116 0)
+			(at 38.481 45.8216 0)
 			(effects
 				(font
@@
 		)
 		(property "Value" "0.1u"
-			(at 25.781 44.323 0)
+			(at 38.481 48.133 0)
 			(effects
 				(font
@@
 		)
 		(property "Footprint" "Capacitor_SMD:C_0805_2012Metric_Pad1.18x1.45mm_HandSolder"
-			(at 23.8252 46.99 0)
+			(at 36.5252 50.8 0)
 			(effects
 				(font
@@
 		)
 		(property "Datasheet" "~"
-			(at 22.86 43.18 0)
+			(at 35.56 46.99 0)
 			(effects
 				(font
@@
 		)
 		(property "Description" ""
-			(at 22.86 43.18 0)
+			(at 35.56 46.99 0)
 			(effects
 				(font
@@
 	(symbol
 		(lib_id "Connector:Micro_SD_Card")
-		(at 78.74 53.34 0)
+		(at 91.44 57.15 0)
 		(unit 1)
 		(exclude_from_sim no)
@@
 		(fields_autoplaced yes)
 		(property "Reference" "SD1"
-			(at 79.375 34.29 0)
+			(at 92.075 38.1 0)
 			(effects
 				(font
@@
 		)
 		(property "Value" "Micro SD"
-			(at 79.375 36.83 0)
+			(at 92.075 40.64 0)
 			(effects
 				(font
@@
 		)
 		(property "Footprint" "LIBS:Medved_SD_Card"
-			(at 107.95 45.72 0)
+			(at 120.65 49.53 0)
 			(effects
 				(font
@@
 		)
 		(property "Datasheet" "http://katalog.we-online.de/em/datasheet/693072010801.pdf"
-			(at 78.74 53.34 0)
+			(at 91.44 57.15 0)
 			(effects
 				(font
@@
 		)
 		(property "Description" ""
-			(at 78.74 53.34 0)
-			(effects
-				(font
+			(at 91.44 57.15 0)
+			(effects
+				(font

Commit message: Updated HW
Parts:
- C3: renamed from C18; footprint Capacitor_SMD:C_0805_2012Metric_Pad1.18x1.45mm_HandSolder -> LIBS:Medved_C_0805
Changed lines of the file:
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@@
 		(comment 1 "https://github.com/xtremespb/frank2")
+	)
+	(junction
+		(at 43.18 57.15)
+		(diameter 0)
+		(color 0 0 0 0)
 	)
 	(no_connect
@@
 	(wire
 		(pts
+			(xy 43.18 57.15) (xy 68.58 57.15)
+		)
+		(stroke
+			(width 0)
+			(type default)
+		)
+	)
+	(wire
+		(pts
 			(xy 55.88 52.07) (xy 68.58 52.07)
 		)
@@
 	(wire
 		(pts
-			(xy 35.56 57.15) (xy 68.58 57.15)
+			(xy 35.56 57.15) (xy 43.18 57.15)
 		)
 		(stroke
@@
 			(font
 				(size 2.54 2.54)
-			)
-			(justify left bottom)
-		)
-	)
-	(label "+3V3"
-		(at 62.23 57.15 0)
-		(fields_autoplaced yes)
-		(effects
-			(font
-				(size 1.27 1.27)
 			)
 			(justify left bottom)
@@
 		(dnp no)
 		(fields_autoplaced yes)
-		(property "Reference" "#PWR036"
+		(property "Reference" "#PWR015"
 			(at 35.56 77.47 0)
 			(effects
@@
 			(project "frank2"
 				(path "/8c0b3d8b-46d3-4173-ab1e-a61765f77d61/1910744e-2d47-4355-a4aa-76cd3c94388f"
-					(reference "#PWR036")
+					(reference "#PWR015")
 					(unit 1)
 				)
@@
 		(on_board yes)
 		(dnp no)
-		(property "Reference" "#PWR035"
+		(property "Reference" "#PWR014"
 			(at 35.56 36.83 0)
 			(effects
@@
 			(project "frank2"
 				(path "/8c0b3d8b-46d3-4173-ab1e-a61765f77d61/1910744e-2d47-4355-a4aa-76cd3c94388f"
-					(reference "#PWR035")
+					(reference "#PWR014")
 					(unit 1)
 				)
@@
 		(on_board yes)
 		(dnp no)
-		(property "Reference" "C18"
+		(property "Reference" "C3"
 			(at 38.481 45.8216 0)
 			(effects
@@
 			)
 		)
-		(property "Footprint" "Capacitor_SMD:C_0805_2012Metric_Pad1.18x1.45mm_HandSolder"
+		(property "Footprint" "LIBS:Medved_C_0805"
 			(at 36.5252 50.8 0)
 			(effects
@@
 			(project "frank2"
 				(path "/8c0b3d8b-46d3-4173-ab1e-a61765f77d61/1910744e-2d47-4355-a4aa-76cd3c94388f"
-					(reference "C18")
+					(reference "C3")
 					(unit 1)
 				)
+			)
+		)
+	)
+	(symbol
+		(lib_id "power:+3V3")
+		(at 43.18 57.15 0)
+		(unit 1)
+		(exclude_from_sim no)
+		(in_bom yes)
+		(on_board yes)
+		(dnp no)
+		(fields_autoplaced yes)
+		(property "Reference" "#PWR063"
+			(at 43.18 60.96 0)
+			(effects
+				(font
+					(size 1.27 1.27)
+				)
+				(hide yes)
+			)
+		)
+		(property "Value" "+3V3"
+			(at 43.18 52.07 0)
+			(effects
+				(font
+					(size 1.27 1.27)
+				)
+			)
+		)
+		(property "Footprint" ""
+			(at 43.18 57.15 0)
+			(effects
+				(font
+					(size 1.27 1.27)
+				)
+				(hide yes)
+			)
+		)
+		(property "Datasheet" ""
+			(at 43.18 57.15 0)
+			(effects
+				(font
+					(size 1.27 1.27)
+				)
+				(hide yes)
+			)
+		)
+		(property "Description" "Power symbol creates a global label with name \"+3V3\""
+			(at 43.18 57.15 0)
+			(effects
+				(font
+					(size 1.27 1.27)
+				)
+				(hide yes)
+			)
+		)
+		(pin "1"
+		)
+		(instances
+			(project ""
+				(path "/8c0b3d8b-46d3-4173-ab1e-a61765f77d61/1910744e-2d47-4355-a4aa-76cd3c94388f"
+					(reference "#PWR063")
+					(unit 1)
+				)

Commit message: HW Rev 2.0
Other:
- title: FRANK2 -> FRANK
Changed lines of the file:
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@@
 	(paper "A4")
 	(title_block
-		(title "FRANK2")
-		(date "2024-11-21")
-		(rev "1.0")
+		(title "FRANK")
+		(date "2024-12-15")
+		(rev "2.0")
 		(company "Mikhail Matveev")
 		(comment 1 "https://github.com/xtremespb/frank2")
