File: usbstack.kicad_sch (KiCad schematic)
At the start: 7 parts

Commit message: HW Rev 2.0
Other:
- title: USB to PS/2 Adapter -> FRANK
Changed lines of the file:
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@@
 	(generator "eeschema")
 	(generator_version "8.0")
-	(paper "A3")
+	(paper "A4")
 	(title_block
-		(title "USB to PS/2 Adapter")
-		(date "2024-12-07")
-		(rev "1.2")
+		(title "FRANK")
+		(date "2024-12-15")
+		(rev "2.0")
 		(company "Mikhail Matveev")
+		(comment 1 "https://github.com/xtremespb/frank2")
 	)
 	(junction
